Commit message: Update physicar body mesh and add detail meshes with textures

File: deepracer_simulation_environment/share/deepracer_simulation_environment/urdf/physicar/physicar_single_cam.urdf (robot description, URDF)
Before this commit: robot physicar_single_cam, 12 links, 11 joints
Links:
- link chassis: geometry visual mesh filename=package://deepracer_simulation_environment/meshes/physicar/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; visual mesh filename=package://deepracer_simulation_environment/meshes/physicar/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
- link servo_pan_link: geometry 

File: deepracer_simulation_environment/share/deepracer_simulation_environment/urdf/physicar/physicar_single_cam_lidar.urdf (robot description, URDF)
Before this commit: robot physicar_single_cam_lidar, 13 links, 12 joints
Links:
- link chassis: geometry visual mesh filename=package://deepracer_simulation_environment/meshes/physicar/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; visual mesh filename=package://deepracer_simulation_environment/meshes/physicar/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
- link servo_pan_link: geometry 
